File: DMH_Tripple_VCA_PCB_1/VCA_C.kicad_sch (KiCad schematic)
At the start: 19 parts, among them Q5 BC548, Q6 BC548, U2 TL074

Commit message: Changed R14 R29 R44 to 100k
Parts:
- R44: value 82k -> 100k
Changed lines of the file:
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@@
 			)
 		)
-		(property "Value" "82k"
+		(property "Value" "100k"
 			(at 87.63 135.89 90)
 			(effects
