File: DMH_Tripple_VCA_PCB_1/DMH_Tripple_VCA_PCB_1.kicad_pcb (KiCad board)
At the start: 2 copper layers, 48 x 175 mm, 88 parts, among them J1 TS_Jack_6.35mm_Sw, J10 TS_Jack_6.35mm_Sw, J100 IDC_02x05, J2 TS_Jack_6.35mm_Sw, J200 IDC_02x05, J3 TS_Jack_6.35mm_Sw, J4 TS_Jack_6.35mm_Sw, J5 TS_Jack_6.35mm_Sw, J50 Conn_01x06, J6 TS_Jack_6.35mm_Sw, J60 Conn_01x06, J7 TS_Jack_6.35mm_Sw, J70 Conn_01x06, J8 TS_Jack_6.35mm_Sw, J9 TS_Jack_6.35mm_Sw, Q1 BC548, Q2 BC548, Q3 BC548, Q4 BC548, Q5 BC548, Q6 BC548, U1 TL074, U2 TL074

Commit message: Changed R14 R29 R44 to 100k
Parts:
- R14, R29, R44: value 82k -> 100k
Changed lines of the file:
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@@
 			)
 		)
-		(property "Value" "82k"
+		(property "Value" "100k"
 			(at 1.27 -2.37 0)
 			(layer "B.Fab")
@@
 			)
 		)
-		(property "Value" "82k"
+		(property "Value" "100k"
 			(at 1.27 -2.37 0)
 			(layer "B.Fab")
@@
 			)
 		)
-		(property "Value" "82k"
+		(property "Value" "100k"
 			(at 1.27 -2.37 0)
 			(layer "B.Fab")

Commit message: Generated Gerbers
Other:
- board text added: "Mk1.0 - March 2025"
- board text removed: "Mk1.0 - Month Year"
Changed lines of the file:
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@@
 			(plot_on_all_layers_selection 0x00000000_00000000_00000000_00000000)
 			(disableapertmacros no)
-			(usegerberextensions no)
+			(usegerberextensions yes)
 			(usegerberattributes yes)
 			(usegerberadvancedattributes yes)
@@
 			(sketchdnponfab yes)
 			(crossoutdnponfab yes)
-			(subtractmaskfromsilk no)
+			(subtractmaskfromsilk yes)
 			(outputformat 1)
 			(mirror no)
-			(drillshape 1)
+			(drillshape 0)
 			(scaleselection 1)
-			(outputdirectory "")
+			(outputdirectory "Gerbers/")
 		)
 	)
@@
 	)
 	(gr_rect
-		(start 54.5 213.25)
-		(end 64.5 215.25)
+		(start 54.8 213.25)
+		(end 64.8 215.25)
 		(stroke
 			(width 0.1)
@@
 		(layer "User.9")
 	)
-	(gr_text "Mk1.0 - Month Year"
-		(at 59.25 216.25 0)
+	(gr_text "Mk1.0 - March 2025"
+		(at 59.55 216.25 0)
 		(layer "B.SilkS")
 		(effects
