File: DMH_Tripple_VCA_PCB_1/Mixer.kicad_sch (KiCad schematic)
At the start: 8 parts, among them U2 TL074

Commit message: Fixed another mistake
U2C and U2D + and - inputs were inverted
Connections:
- net GND: now also U2.10 (+), U2.12 (+); no longer U2.13 (-), U2.9 (-)
- net at R46.2, R47.1, R48.2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: now also U2.9 (-); no longer U2.10 (+)
- net at R50.2, R51.1: now also U2.13 (-); no longer U2.12 (+)
Changed lines of the file:
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@@
 		(lib_id "Amplifier_Operational:TL074")
 		(at 76.2 88.9 0)
+		(mirror x)
 		(unit 3)
 		(exclude_from_sim no)
@@
 		(on_board yes)
 		(dnp no)
-		(fields_autoplaced yes)
 		(property "Reference" "U2"
-			(at 76.2 78.74 0)
+			(at 76.2 99.06 0)
 			(effects
 				(font
@@
 		)
 		(property "Value" "TL074"
-			(at 76.2 81.28 0)
+			(at 76.2 96.52 0)
 			(effects
 				(font
@@
 		)
 		(property "Footprint" "Package_DIP:DIP-14_W7.62mm_Socket"
-			(at 74.93 86.36 0)
+			(at 74.93 91.44 0)
 			(effects
 				(font
@@
 		)
 		(property "Datasheet" "http://www.ti.com/lit/ds/symlink/tl071.pdf"
-			(at 77.47 83.82 0)
+			(at 77.47 93.98 0)
 			(effects
 				(font
@@
 		(lib_id "Amplifier_Operational:TL074")
 		(at 114.3 91.44 0)
+		(mirror x)
 		(unit 4)
 		(exclude_from_sim no)
@@
 		(on_board yes)
 		(dnp no)
-		(fields_autoplaced yes)
 		(property "Reference" "U2"
-			(at 114.3 81.28 0)
+			(at 114.3 101.6 0)
 			(effects
 				(font
@@
 		)
 		(property "Value" "TL074"
-			(at 114.3 83.82 0)
+			(at 114.3 99.06 0)
 			(effects
 				(font
@@
 		)
 		(property "Footprint" "Package_DIP:DIP-14_W7.62mm_Socket"
-			(at 113.03 88.9 0)
+			(at 113.03 93.98 0)
 			(effects
 				(font
@@
 		)
 		(property "Datasheet" "http://www.ti.com/lit/ds/symlink/tl071.pdf"
-			(at 115.57 86.36 0)
-			(effects
-				(font
+			(at 115.57 96.52 0)
+			(effects
+				(font
